File: Driver.sch (KiCad schematic (older format))
At the start: 31 parts, among them J13 CONN_01X10, J14 CONN_01X10, J15 CONN_01X01, J16 CONN_01X01, J17 CONN_01X01, J18 CONN_01X01, Q2 PSMN1R0-40YLD, Q4 PSMN1R0-40YLD, Q5 PSMN1R0-40YLD, Q7 PSMN1R0-40YLD, U4 A4957, U5 ACS722

Commit message: FETがパラになったｗｗｗ
Parts:
- added Q? (x4): PSMN1R0-40YLD, SMD_Packages:LFPAK56_SO8_SOT1023, symbol PSMN1R0-40YLD
- added R? (x4): 10, Resistors_SMD:R_0603, symbol R
- added R? (x4): 10k, Resistors_SMD:R_0603, symbol R
Connections:
- net GND: now also Q?.1 (S), Q?.1 (S), Q?.2 (S), Q?.2 (S), Q?.3 (S), Q?.3 (S), R?.1, R?.2
- net V_BATT: now also Q?.5 (D), Q?.5 (D)
- net at Q2.1 (S), Q2.2 (S), Q2.3 (S)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: now also Q?.1 (S), Q?.2 (S), Q?.3 (S), Q?.5 (D), R?.1
- net at Q2.4 (G), R23.2: now also R21.2; no longer R21.1
- net at Q7.4 (G), R34.2: now also R32.2; no longer R32.1
- net at C29.2, J17.1 (P1), Q4.1 (S)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: now also Q?.1 (S), Q?.2 (S), Q?.3 (S), Q?.5 (D), R?.2
- net at Q4.4 (G), R25.1: now also R27.1; no longer R27.2
- net at Q5.4 (G), R26.1: now also R28.1; no longer R28.2
- net at U4.18 (GLB): now also R28.2, R?.2; no longer R28.1
- net at U4.20 (GHB): now also R27.2, R?.2; no longer R27.1
- net at U4.24 (GHA): now also R21.1, R?.1; no longer R21.2
- net at C21.2, U4.2 (GLA): now also R32.1, R?.1; no longer R32.2
- new net: Q?.4 (G), R?.1, R?.1 (x2)
- new net: Q?.4 (G), R?.2, R?.2 (x2)
Other:
- moved on the sheet: C23, J13, J14, J15, J17, J18, JP1, Q3, Q4, Q5, R21, R22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

Commit message: しんちょく
Parts:
- gave numbers to parts that had none: 12
Changed lines of the file:
@@
 $EndComp
 $Comp
-L R R?
+L R R46
 U 1 1 58CF16FF
 P 9150 3100
-F 0 "R?" V 9230 3100 50  0000 C CNN
+AR Path="/58CBAEB3/58CF16FF" Ref="R46"  Part="1"
+AR Path="/58CBB47A/58CF16FF" Ref="R54"  Part="1"
+F 0 "R46" V 9230 3100 50  0000 C CNN
 F 1 "10" V 9150 3100 50  0000 C CNN
 F 2 "Resistors_SMD:R_0603" V 9080 3100 50  0001 C CNN
@@
 $EndComp
 $Comp
-L R R?
+L R R44
 U 1 1 58CF17B1
 P 9000 3100
-F 0 "R?" V 9080 3100 50  0000 C CNN
+AR Path="/58CBAEB3/58CF17B1" Ref="R44"  Part="1"
+AR Path="/58CBB47A/58CF17B1" Ref="R52"  Part="1"
+F 0 "R44" V 9080 3100 50  0000 C CNN
 F 1 "10k" V 9000 3100 50  0000 C CNN
 F 2 "Resistors_SMD:R_0603" V 8930 3100 50  0001 C CNN
@@
 $EndComp
 $Comp
-L PSMN1R0-40YLD Q?
+L PSMN1R0-40YLD Q13
 U 1 1 58CF1D35
 P 8600 2900
-F 0 "Q?" H 8400 3200 50  0000 L CNN
+AR Path="/58CBAEB3/58CF1D35" Ref="Q13"  Part="1"
+AR Path="/58CBB47A/58CF1D35" Ref="Q17"  Part="1"
+F 0 "Q13" H 8400 3200 50  0000 L CNN
 F 1 "PSMN1R0-40YLD" H 8400 2650 50  0000 L CNN
 F 2 "SMD_Packages:LFPAK56_SO8_SOT1023" H 8600 3100 50  0001 C CIN
@@
 $EndComp
 $Comp
-L R R?
+L R R45
 U 1 1 58CF8994
 P 9000 4150
-F 0 "R?" V 9080 4150 50  0000 C CNN
+AR Path="/58CBAEB3/58CF8994" Ref="R45"  Part="1"
+AR Path="/58CBB47A/58CF8994" Ref="R53"  Part="1"
+F 0 "R45" V 9080 4150 50  0000 C CNN
 F 1 "10" V 9000 4150 50  0000 C CNN
 F 2 "Resistors_SMD:R_0603" V 8930 4150 50  0001 C CNN
@@
 $EndComp
 $Comp
-L R R?
+L R R43
 U 1 1 58CF8A37
 P 8850 4150
-F 0 "R?" V 8930 4150 50  0000 C CNN
+AR Path="/58CBAEB3/58CF8A37" Ref="R43"  Part="1"
+AR Path="/58CBB47A/58CF8A37" Ref="R51"  Part="1"
+F 0 "R43" V 8930 4150 50  0000 C CNN
 F 1 "10k" V 8850 4150 50  0000 C CNN
 F 2 "Resistors_SMD:R_0603" V 8780 4150 50  0001 C CNN
@@
 $EndComp
 $Comp
-L PSMN1R0-40YLD Q?
+L PSMN1R0-40YLD Q12
 U 1 1 58CF9E77
 P 8450 4000
-F 0 "Q?" H 8250 4300 50  0000 L CNN
+AR Path="/58CBAEB3/58CF9E77" Ref="Q12"  Part="1"
+AR Path="/58CBB47A/58CF9E77" Ref="Q16"  Part="1"
+F 0 "Q12" H 8250 4300 50  0000 L CNN
 F 1 "PSMN1R0-40YLD" H 8250 3750 50  0000 L CNN
 F 2 "SMD_Packages:LFPAK56_SO8_SOT1023" H 8450 4200 50  0001 C CIN
@@
 $EndComp
 $Comp
-L PSMN1R0-40YLD Q?
+L PSMN1R0-40YLD Q10
 U 1 1 58CFFD18
 P 7750 4000
-F 0 "Q?" H 7550 4300 50  0000 L CNN
+AR Path="/58CBAEB3/58CFFD18" Ref="Q10"  Part="1"
+AR Path="/58CBB47A/58CFFD18" Ref="Q14"  Part="1"
+F 0 "Q10" H 7550 4300 50  0000 L CNN
 F 1 "PSMN1R0-40YLD" H 7550 3750 50  0000 L CNN
 F 2 "SMD_Packages:LFPAK56_SO8_SOT1023" H 7750 4200 50  0001 C CIN
@@
 $EndComp
 $Comp
-L R R?
+L R R41
 U 1 1 58D006F8
 P 7350 4150
-F 0 "R?" V 7430 4150 50  0000 C CNN
+AR Path="/58CBAEB3/58D006F8" Ref="R41"  Part="1"
+AR Path="/58CBB47A/58D006F8" Ref="R49"  Part="1"
+F 0 "R41" V 7430 4150 50  0000 C CNN
 F 1 "10k" V 7350 4150 50  0000 C CNN
 F 2 "Resistors_SMD:R_0603" V 7280 4150 50  0001 C CNN
@@
 $EndComp
 $Comp
-L R R?
+L R R39
 U 1 1 58D008FF
 P 7200 4150
-F 0 "R?" V 7280 4150 50  0000 C CNN
+AR Path="/58CBAEB3/58D008FF" Ref="R39"  Part="1"
+AR Path="/58CBB47A/58D008FF" Ref="R47"  Part="1"
+F 0 "R39" V 7280 4150 50  0000 C CNN
 F 1 "10" V 7200 4150 50  0000 C CNN
 F 2 "Resistors_SMD:R_0603" V 7130 4150 50  0001 C CNN
@@
 $EndComp
 $Comp
-L PSMN1R0-40YLD Q?
+L PSMN1R0-40YLD Q11
 U 1 1 58D053B7
 P 7900 2900
-F 0 "Q?" H 7700 3200 50  0000 L CNN
+AR Path="/58CBAEB3/58D053B7" Ref="Q11"  Part="1"
+AR Path="/58CBB47A/58D053B7" Ref="Q15"  Part="1"
+F 0 "Q11" H 7700 3200 50  0000 L CNN
 F 1 "PSMN1R0-40YLD" H 7700 2650 50  0000 L CNN
 F 2 "SMD_Packages:LFPAK56_SO8_SOT1023" H 7900 3100 50  0001 C CIN
@@
 $EndComp
 $Comp
-L R R?
+L R R42
 U 1 1 58D057CC
 P 7450 3100
-F 0 "R?" V 7530 3100 50  0000 C CNN
+AR Path="/58CBAEB3/58D057CC" Ref="R42"  Part="1"
+AR Path="/58CBB47A/58D057CC" Ref="R50"  Part="1"
+F 0 "R42" V 7530 3100 50  0000 C CNN
 F 1 "10k" V 7450 3100 50  0000 C CNN
 F 2 "Resistors_SMD:R_0603" V 7380 3100 50  0001 C CNN
@@
 $EndComp
 $Comp
-L R R?
+L R R40
 U 1 1 58D05888
 P 7300 3100
-F 0 "R?" V 7380 3100 50  0000 C CNN
+AR Path="/58CBAEB3/58D05888" Ref="R40"  Part="1"
+AR Path="/58CBB47A/58D05888" Ref="R48"  Part="1"
+F 0 "R40" V 7380 3100 50  0000 C CNN
 F 1 "10" V 7300 3100 50  0000 C CNN
 F 2 "Resistors_SMD:R_0603" V 7230 3100 50  0001 C CNN

Commit message: しんちょく
Parts:
- renumbered C29 to C22, J14 to J13, J13 to J14, J16 to J15, J15 to J16, Q7 to Q2, Q2 to Q3, Q10 to Q4, Q11 to Q5, Q12 to Q6, Q13 to Q7, Q5 to Q8, Q4 to Q9, R32 to R22, R34 to R24, R39 to R25, R40 to R26, R41 to R27, R42 to R28, R43 to R29, R44 to R30, R45 to R31, R46 to R32, R26 to R33, R25 to R34, R28 to R35, R27 to R36

Commit message: 進捗セーブ
Parts:
- J15, J16, J17, J18: footprint Mounting_Holes:MountingHole_3mm_Pad_Via -> Mounting_Holes:MountingHole_2.7mm_Pad_Via

Commit message: 進捗セーブ
Connections:
- net +3V3: now also J14.5 (P5); no longer J14.8 (P8)
- net GND: now also J14.3 (P3); no longer J14.10 (P10)
- net V_BATT: now also J14.2 (P2); no longer J14.1 (P1)
- net at U5.7 (VIOUT): now also J14.1 (P1); no longer J14.9 (P9)
- net at Q2.5 (D), Q3.1 (S), Q3.2 (S)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: now also C22.2, U4.19 (SB); no longer U4.1 (SA)
- net at J17.1 (P1), Q6.5 (D), Q7.1 (S)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: now also C21.2, U4.1 (SA); no longer C22.2, U4.19 (SB)
- net at R31.2, R35.2: now also U4.2 (GLA); no longer U4.18 (GLB)
- net at R32.2, R36.2: now also U4.24 (GHA); no longer U4.20 (GHB)
- net at R21.1, R26.1: now also U4.20 (GHB); no longer U4.24 (GHA)
- net at R22.1, R25.1: now also U4.18 (GLB); no longer C21.2, U4.2 (GLA)
Other:
- moved on the sheet: J20

Commit message: 一度全部配線はできた，きれいにする必要あり
Parts:
- removed J13: CONN_01X10, Pin_Headers:Pin_Header_Straight_1x10_Pitch2.00mm_SMD_Pin1Left, symbol CONN_01X10
Connections:
- net at J14.10 (P10): now also U4.8 (BLO)
- net at J14.4 (P4): now also U4.16 (RESET)
- net at J14.6 (P6): now also R19.2, U4.15 (FAULT)
- net at J14.7 (P7): now also U4.11 (AHI)
- net at J14.8 (P8): now also U4.10 (ALO)
- net at J14.9 (P9): now also U4.9 (BHI)
- no-connect marks 8 -> 0
