File: Driver.sch (KiCad schematic (older format))
At the start: 42 parts, among them J14 CONN_01X10, J15 CONN_01X01, J16 CONN_01X01, J17 CONN_01X01, J18 CONN_01X01, Q2 PSMN1R0-40YLD, Q3 PSMN1R0-40YLD, Q4 PSMN1R0-40YLD, Q5 PSMN1R0-40YLD, Q6 PSMN1R0-40YLD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

Commit message: アノテーション前のセーブ
Parts:
- C32: renamed from C?; footprint (none) -> Capacitors_SMD:C_0603
- U7: renamed from U?; footprint (none) -> Housings_DFN_QFN:QFN-12_3x3mm_Pitch0.5mm_With_Fused_Sensed_Current_Loop

Commit message: 進捗，セーブ
Parts:
- added C33, C34, C35: C, Capacitors_SMD:C_0603, symbol C
Connections:
- net GND: now also C33.2, C34.2, C35.2
- net V_BATT: now also C33.1, C34.1, C35.1
