File: Driver.sch (KiCad schematic (older format))
At the start: 45 parts, among them J14 CONN_01X10, J15 CONN_01X01, J16 CONN_01X01, J17 CONN_01X01, J18 CONN_01X01, Q2 PSMN1R0-40YLD, Q3 PSMN1R0-40YLD, Q4 PSMN1R0-40YLD, Q5 PSMN1R0-40YLD, Q6 PSMN1R0-40YLD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

Commit message: 470uだったのところを470nに修正 ネットリスト変更して再アノテーションした ピンソケットとピンヘッダ以外のBOMだしおわり
Parts:
- C19: value 470u -> 470n
Changed lines of the file:
@@
 AR Path="/58CBB47A/58CC7521" Ref="C26"  Part="1"
 F 0 "C26" H 4325 2000 50  0000 L CNN
-F 1 "470u" H 4325 1800 50  0000 L CNN
+F 1 "470n" H 4325 1800 50  0000 L CNN
 F 2 "Capacitors_SMD:C_0603" H 4338 1750 50  0001 C CNN
 F 3 "" H 4300 1900 50  0001 C CNN

Commit message: ブートストラップコンデンサの値を決めた
Parts:
- C20: value 5.66u -> 4.4u
- C21, C22: value 0.283u -> 0.22u
Changed lines of the file:
@@
 $Descr A4 11693 8268
 encoding utf-8
-Sheet 4 5
+Sheet 5 5
 Title ""
 Date ""
@@
 AR Path="/58CBB47A/58CC7357" Ref="C27"  Part="1"
 F 0 "C27" H 4725 2500 50  0000 L CNN
-F 1 "5.66u" H 4725 2300 50  0000 L CNN
+F 1 "4.4u" H 4725 2300 50  0000 L CNN
 F 2 "Capacitors_SMD:C_0805" H 4738 2250 50  0001 C CNN
 F 3 "" H 4700 2400 50  0001 C CNN
@@
 AR Path="/58CBB47A/58CCC902" Ref="C28"  Part="1"
 F 0 "C28" H 5175 2950 50  0000 L CNN
-F 1 "0.283u" H 5175 2750 50  0000 L CNN
+F 1 "0.22u" H 5175 2750 50  0000 L CNN
 F 2 "Capacitors_SMD:C_0603" H 5188 2700 50  0001 C CNN
 F 3 "" H 5150 2850 50  0001 C CNN
@@
 AR Path="/58CBB47A/58CCCAD7" Ref="C29"  Part="1"
 F 0 "C29" H 5175 3700 50  0000 L CNN
-F 1 "0.283u" H 5175 3500 50  0000 L CNN
+F 1 "0.22u" H 5175 3500 50  0000 L CNN
 F 2 "Capacitors_SMD:C_0603" H 5188 3450 50  0001 C CNN
 F 3 "" H 5150 3600 50  0001 C CNN
