File: _saved_Driver.sch (KiCad schematic (older format))
At the start: 42 parts, among them J14 CONN_01X10, J15 CONN_01X01, J16 CONN_01X01, J17 CONN_01X01, J18 CONN_01X01, Q2 PSMN1R0-40YLD, Q3 PSMN1R0-40YLD, Q4 PSMN1R0-40YLD, Q5 PSMN1R0-40YLD, Q6 PSMN1R0-40YLD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

Commit message: しんちょくセーブ
Parts:
- C32: renamed from C?; footprint (none) -> Capacitors_SMD:C_0603
- U7: renamed from U?; footprint (none) -> Housings_DFN_QFN:QFN-12_3x3mm_Pitch0.5mm_With_Fused_Sensed_Current_Loop
Changed lines of the file:
@@
 $EndDescr
 $Comp
-L GND #PWR049
+L GND #PWR048
 U 1 1 58CBF233
 P 2700 5200
-AR Path="/58CBAEB3/58CBF233" Ref="#PWR049"  Part="1"
-AR Path="/58CBB47A/58CBF233" Ref="#PWR061"  Part="1"
-F 0 "#PWR061" H 2700 4950 50  0001 C CNN
+AR Path="/58CBAEB3/58CBF233" Ref="#PWR048"  Part="1"
+AR Path="/58CBB47A/58CBF233" Ref="#PWR058"  Part="1"
+F 0 "#PWR058" H 2700 4950 50  0001 C CNN
 F 1 "GND" H 2700 5050 50  0000 C CNN
 F 2 "" H 2700 5200 50  0001 C CNN
@@
 $EndComp
 $Comp
-L +3V3 #PWR051
+L +3V3 #PWR049
 U 1 1 58CBF5F4
 P 2700 5400
-AR Path="/58CBAEB3/58CBF5F4" Ref="#PWR051"  Part="1"
-AR Path="/58CBB47A/58CBF5F4" Ref="#PWR063"  Part="1"
-F 0 "#PWR063" H 2700 5250 50  0001 C CNN
+AR Path="/58CBAEB3/58CBF5F4" Ref="#PWR049"  Part="1"
+AR Path="/58CBB47A/58CBF5F4" Ref="#PWR059"  Part="1"
+F 0 "#PWR059" H 2700 5250 50  0001 C CNN
 F 1 "+3V3" H 2700 5540 50  0000 C CNN
 F 2 "" H 2700 5400 50  0001 C CNN
@@
 V_BATT
 $Comp
-L GND #PWR052
+L GND #PWR050
 U 1 1 58CC090D
 P 7450 4400
-AR Path="/58CBAEB3/58CC090D" Ref="#PWR052"  Part="1"
-AR Path="/58CBB47A/58CC090D" Ref="#PWR064"  Part="1"
-F 0 "#PWR064" H 7450 4150 50  0001 C CNN
+AR Path="/58CBAEB3/58CC090D" Ref="#PWR050"  Part="1"
+AR Path="/58CBB47A/58CC090D" Ref="#PWR060"  Part="1"
+F 0 "#PWR060" H 7450 4150 50  0001 C CNN
 F 1 "GND" H 7450 4250 50  0000 C CNN
 F 2 "" H 7450 4400 50  0001 C CNN
@@
 $EndComp
 $Comp
-L GND #PWR053
+L GND #PWR051
 U 1 1 58CC5771
 P 2900 2850
-AR Path="/58CBAEB3/58CC5771" Ref="#PWR053"  Part="1"
-AR Path="/58CBB47A/58CC5771" Ref="#PWR065"  Part="1"
-F 0 "#PWR065" H 2900 2600 50  0001 C CNN
+AR Path="/58CBAEB3/58CC5771" Ref="#PWR051"  Part="1"
+AR Path="/58CBB47A/58CC5771" Ref="#PWR061"  Part="1"
+F 0 "#PWR061" H 2900 2600 50  0001 C CNN
 F 1 "GND" H 2900 2700 50  0000 C CNN
 F 2 "" H 2900 2850 50  0001 C CNN
@@
 $EndComp
 $Comp
-L +3V3 #PWR054
+L +3V3 #PWR052
 U 1 1 58CC5AE0
 P 3200 2750
-AR Path="/58CBAEB3/58CC5AE0" Ref="#PWR054"  Part="1"
-AR Path="/58CBB47A/58CC5AE0" Ref="#PWR066"  Part="1"
-F 0 "#PWR066" H 3200 2600 50  0001 C CNN
+AR Path="/58CBAEB3/58CC5AE0" Ref="#PWR052"  Part="1"
+AR Path="/58CBB47A/58CC5AE0" Ref="#PWR062"  Part="1"
+F 0 "#PWR062" H 3200 2600 50  0001 C CNN
 F 1 "+3V3" H 3200 2890 50  0000 C CNN
 F 2 "" H 3200 2750 50  0001 C CNN
@@
 $EndComp
 $Comp
-L GND #PWR055
+L GND #PWR053
 U 1 1 58CC6C27
 P 4150 4500
-AR Path="/58CBAEB3/58CC6C27" Ref="#PWR055"  Part="1"
-AR Path="/58CBB47A/58CC6C27" Ref="#PWR067"  Part="1"
-F 0 "#PWR067" H 4150 4250 50  0001 C CNN
+AR Path="/58CBAEB3/58CC6C27" Ref="#PWR053"  Part="1"
+AR Path="/58CBB47A/58CC6C27" Ref="#PWR063"  Part="1"
+F 0 "#PWR063" H 4150 4250 50  0001 C CNN
 F 1 "GND" H 4150 4350 50  0000 C CNN
 F 2 "" H 4150 4500 50  0001 C CNN
@@
 $EndComp
 $Comp
-L GND #PWR056
+L GND #PWR054
 U 1 1 58CC74DF
 P 4850 2400
-AR Path="/58CBAEB3/58CC74DF" Ref="#PWR056"  Part="1"
-AR Path="/58CBB47A/58CC74DF" Ref="#PWR068"  Part="1"
-F 0 "#PWR068" H 4850 2150 50  0001 C CNN
+AR Path="/58CBAEB3/58CC74DF" Ref="#PWR054"  Part="1"
+AR Path="/58CBB47A/58CC74DF" Ref="#PWR064"  Part="1"
+F 0 "#PWR064" H 4850 2150 50  0001 C CNN
 F 1 "GND" H 4850 2250 50  0000 C CNN
 F 2 "" H 4850 2400 50  0001 C CNN
@@
 $EndComp
 $Comp
-L GND #PWR057
+L GND #PWR055
 U 1 1 58CC7D18
 P 3550 2350
-AR Path="/58CBAEB3/58CC7D18" Ref="#PWR057"  Part="1"
-AR Path="/58CBB47A/58CC7D18" Ref="#PWR069"  Part="1"
-F 0 "#PWR069" H 3550 2100 50  0001 C CNN
+AR Path="/58CBAEB3/58CC7D18" Ref="#PWR055"  Part="1"
+AR Path="/58CBB47A/58CC7D18" Ref="#PWR065"  Part="1"
+F 0 "#PWR065" H 3550 2100 50  0001 C CNN
 F 1 "GND" H 3550 2200 50  0000 C CNN
 F 2 "" H 3550 2350 50  0001 C CNN
@@
 $EndComp
 $Comp
-L GND #PWR058
+L GND #PWR056
 U 1 1 58CD0C8C
 P 10250 4900
-AR Path="/58CBAEB3/58CD0C8C" Ref="#PWR058"  Part="1"
-AR Path="/58CBB47A/58CD0C8C" Ref="#PWR070"  Part="1"
-F 0 "#PWR070" H 10250 4650 50  0001 C CNN
+AR Path="/58CBAEB3/58CD0C8C" Ref="#PWR056"  Part="1"
+AR Path="/58CBB47A/58CD0C8C" Ref="#PWR066"  Part="1"
+F 0 "#PWR066" H 10250 4650 50  0001 C CNN
 F 1 "GND" H 10250 4750 50  0000 C CNN
 F 2 "" H 10250 4900 50  0001 C CNN
@@
 $EndComp
 $Comp
-L +3V3 #PWR059
+L +3V3 #PWR057
 U 1 1 58CD1628
 P 10850 4900
-AR Path="/58CBAEB3/58CD1628" Ref="#PWR059"  Part="1"
-AR Path="/58CBB47A/58CD1628" Ref="#PWR071"  Part="1"
-F 0 "#PWR071" H 10850 4750 50  0001 C CNN
+AR Path="/58CBAEB3/58CD1628" Ref="#PWR057"  Part="1"
+AR Path="/58CBB47A/58CD1628" Ref="#PWR067"  Part="1"
+F 0 "#PWR067" H 10850 4750 50  0001 C CNN
 F 1 "+3V3" H 10850 5040 50  0000 C CNN
 F 2 "" H 10850 4900 50  0001 C CNN
@@
 	2900 3600 3400 3600
 $Comp
-L ACS711 U?
+L ACS711 U7
 U 1 1 58B2E1B0
 P 10600 3950
-F 0 "U?" H 10400 4250 60  0000 C CNN
+AR Path="/58CBB47A/58B2E1B0" Ref="U7"  Part="1"
+AR Path="/58CBAEB3/58B2E1B0" Ref="U5"  Part="1"
+F 0 "U7" H 10400 4250 60  0000 C CNN
 F 1 "ACS711" H 10750 4250 60  0000 C CNN
-F 2 "" H 10600 3950 60  0001 C CNN
+F 2 "Housings_DFN_QFN:QFN-12_3x3mm_Pitch0.5mm_With_Fused_Sensed_Current_Loop" H 10600 3950 60  0001 C CNN
 F 3 "" H 10600 3950 60  0001 C CNN
 	1    10600 3950
@@
 NoConn ~ 10550 4300
 $Comp
-L C C?
+L C C32
 U 1 1 58B31138
 P 10600 4650
-F 0 "C?" H 10625 4750 50  0000 L CNN
+AR Path="/58CBB47A/58B31138" Ref="C32"  Part="1"
+AR Path="/58CBAEB3/58B31138" Ref="C31"  Part="1"
+F 0 "C32" H 10625 4750 50  0000 L CNN
 F 1 "C" H 10625 4550 50  0000 L CNN
-F 2 "" H 10638 4500 50  0001 C CNN
+F 2 "Capacitors_SMD:C_0603" H 10638 4500 50  0001 C CNN
 F 3 "" H 10600 4650 50  0001 C CNN
 	1    10600 4650
