File: nmkgmmd_v10_brd.kicad_pcb (KiCad board)
At the start: 2 copper layers, 66 parts, among them J1 CONN_01X05, J10 CONN_01X10, J11 CONN_01X10, J12 CONN_01X10, J2 CONN_01X03, J3 CONN_01X03, J4 CONN_01X04, J5 CONN_01X04, J6 CONN_01X04, J7 CONN_01X03, J8 CONN_01X03, J9 CONN_01X10, Q1 BSS138PS, SW1 SKRPACE010, SW2 SW_DPDT_x2, U1 STM32F303CCTx, U2 MCP16301, U3 MCP16301, Y1 Crystal

Commit message: 回路図作ってみた
Parts:
- added C17: 0.1u, Capacitors_SMD:C_0603, F.Cu at (170.0, 108.0)
- added C18: 0.1u, Capacitors_SMD:C_0603, F.Cu at (151.2, 92.8)
- added C19: 470u, Capacitors_SMD:C_0603, F.Cu at (167.2, 100.0)
- added C20: 5.66u, Capacitors_SMD:C_0805, F.Cu at (165.0, 112.0)
- added C21: 0.283u, Capacitors_SMD:C_0603, F.Cu at (164.0, 97.0)
- added C22: 0.283u, Capacitors_SMD:C_0603, F.Cu at (165.2, 116.0)
- added C23: 0.1u, Capacitors_SMD:C_0603, B.Cu at (120.2, 73.0)
- added C24: 0.1u, Capacitors_SMD:C_0603, F.Cu at (125.4, 12.5)
- added C25: 0.1u, Capacitors_SMD:C_0603, F.Cu at (111.2, 31.6)
- added C26: 470u, Capacitors_SMD:C_0603, F.Cu at (138.4, 2.48)
- added C27: 5.66u, Capacitors_SMD:C_0805, F.Cu at (116.6, 21.6)
- added C28: 0.283u, Capacitors_SMD:C_0603, F.Cu at (133.5, 2.48)
- added C29: 0.283u, Capacitors_SMD:C_0603, F.Cu at (106.5, 31.6)
- added C30: 0.1u, Capacitors_SMD:C_0603, F.Cu at (132.5, 7.53)
- added D10: D, Diodes_SMD:D_SOD-123, F.Cu at (167.0, 105.0)
- added D11: D, Diodes_SMD:D_SOD-123, F.Cu at (101.1, 31.1)
- added J13: CONN_01X10, Pin_Headers:Pin_Header_Straight_1x10_Pitch2.00mm_SMD_Pin1Left, B.Cu at (130.0, 90.0)
- added J14: CONN_01X10, Pin_Headers:Pin_Header_Straight_1x10_Pitch2.00mm_SMD_Pin1Left, B.Cu at (130.0, 130.0)
- added J15: CONN_01X01, Mounting_Holes:MountingHole_3mm_Pad_Via, F.Cu at (109.0, 122.0)
- added J16: CONN_01X01, Mounting_Holes:MountingHole_3mm_Pad_Via, F.Cu at (109.0, 98.0)
- added J17: CONN_01X01, Mounting_Holes:MountingHole_3mm_Pad_Via, F.Cu at (109.0, 114.0)
- added J18: CONN_01X01, Mounting_Holes:MountingHole_3mm_Pad_Via, F.Cu at (109.0, 106.0)
- added J19: CONN_01X10, Pin_Headers:Pin_Header_Straight_1x10_Pitch2.00mm_SMD_Pin1Left, F.Cu at (79.1, 12.0)
- added J20: CONN_01X10, Pin_Headers:Pin_Header_Straight_1x10_Pitch2.00mm_SMD_Pin1Left, F.Cu at (89.1, 12.0)
- added J21: CONN_01X01, Mounting_Holes:MountingHole_3mm_Pad_Via, F.Cu at (109.2, 24.1)
- added J22: CONN_01X01, Mounting_Holes:MountingHole_3mm_Pad_Via, F.Cu at (125.7, 4.97)
- added J23: CONN_01X01, Mounting_Holes:MountingHole_3mm_Pad_Via, F.Cu at (99.2, 23.1)
- added J24: CONN_01X01, Mounting_Holes:MountingHole_3mm_Pad_Via, F.Cu at (112.4, 14.0)
- added JP1: Jumper_NC_Dual, Connect:GS3, B.Cu at (115.0, 71.0)
- added JP2: Jumper_NC_Dual, Connect:GS3, F.Cu at (89.9, 30.5)
- added Q2: PSMN1R0-40YLD, SMD_Packages:LFPAK56_SO8_SOT1023, F.Cu at (120.0, 107.5)
- added Q3: PSMN1R0-40YLD, SMD_Packages:LFPAK56_SO8_SOT1023, F.Cu at (132.9, 107.5)
- added Q4: PSMN1R0-40YLD, SMD_Packages:LFPAK56_SO8_SOT1023, F.Cu at (120.0, 115.0)
- added Q5: PSMN1R0-40YLD, SMD_Packages:LFPAK56_SO8_SOT1023, F.Cu at (132.9, 115.0)
- added Q6: PSMN1R0-40YLD, SMD_Packages:LFPAK56_SO8_SOT1023, F.Cu at (114.0, 4.47)
- added Q7: PSMN1R0-40YLD, SMD_Packages:LFPAK56_SO8_SOT1023, F.Cu at (100.8, 4.47)
- added Q8: PSMN1R0-40YLD, SMD_Packages:LFPAK56_SO8_SOT1023, F.Cu at (80.6, 28.6)
- added Q9: PSMN1R0-40YLD, SMD_Packages:LFPAK56_SO8_SOT1023, F.Cu at (100.8, 13.5)
- added R19: 10k, Resistors_SMD:R_0603, F.Cu at (158.0, 96.0)
- added R20: 0, Resistors_SMD:R_0603, B.Cu at (158.0, 101.0)
- added R21: 10, Resistors_SMD:R_0603, B.Cu at (125.0, 105.4)
- added R22: 10, Resistors_SMD:R_0603, B.Cu at (138.0, 103.9)
- added R23: 10k, Resistors_SMD:R_0603, B.Cu at (125.0, 103.9)
- added R24: 10k, Resistors_SMD:R_0603, B.Cu at (138.0, 105.4)
- added R25: 10k, Resistors_SMD:R_0603, B.Cu at (125.0, 112.9)
- added R26: 10k, Resistors_SMD:R_0603, B.Cu at (138.0, 112.9)
- added R27: 10, Resistors_SMD:R_0603, B.Cu at (125.0, 111.4)
- added R28: 10, Resistors_SMD:R_0603, B.Cu at (138.0, 111.4)
- added R29: 10k, Resistors_SMD:R_0603, F.Cu at (136.0, 7.47)
- added R30: 0, Resistors_SMD:R_0603, F.Cu at (132.1, 12.5)
- added R31: 10, Resistors_SMD:R_0603, F.Cu at (125.2, 17.5)
- added R32: 10, Resistors_SMD:R_0603, F.Cu at (115.9, 26.8)
- added R33: 10k, Resistors_SMD:R_0603, F.Cu at (120.5, 20.4)
- added R34: 10k, Resistors_SMD:R_0603, F.Cu at (128.8, 12.5)
- added R35: 10k, Resistors_SMD:R_0603, F.Cu at (123.8, 22.5)
- added R36: 10k, Resistors_SMD:R_0603, F.Cu at (128.5, 17.5)
- added R37: 10, Resistors_SMD:R_0603, F.Cu at (119.2, 26.8)
- added R38: 10, Resistors_SMD:R_0603, F.Cu at (114.6, 31.8)
- added U4: A4957, SMD_Packages:Allegro_A4957_QFN-24-1EP_4x4mm_Pitch0.5mm, F.Cu at (147.0, 111.0)
- added U5: ACS722, SMD_Packages:SOIC-8-N, B.Cu at (115.0, 78.0)
- added U6: A4957, SMD_Packages:Allegro_A4957_QFN-24-1EP_4x4mm_Pitch0.5mm, F.Cu at (95.7, 32.5)
- added U7: ACS722, SMD_Packages:SOIC-8-N, F.Cu at (120.5, 14.0)
- moved R1 226.5 mm to (4.43, 37.1)
- moved R2 221.2 mm to (7.38, 37.1)
- moved R7 220.6 mm to (1.48, 37.1)
- moved R3 215.4 mm to (10.4, 37.1)
- moved R11 212.2 mm to (13.6, 37.1)
- moved R4 211.4 mm to (16.8, 37.1)
- moved R6 210.1 mm to (19.9, 37.1)
- moved R5 202.2 mm to (23.0, 37.1)
- moved J9 199.4 mm to (5.03, 3.10)
- moved D1 198.8 mm to (32.5, 36.9)
- moved R9 198.7 mm to (29.4, 37.1)
- moved D2 198.2 mm to (35.9, 36.9)
- moved D4 196.8 mm to (51.6, 22.9)
- moved D5 196.8 mm to (48.3, 22.9)
- moved R10 196.7 mm to (26.2, 37.1)
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Other:
- board outline added: 50 x 50 mm

Commit message: しんちょく
Parts:
- added Q10: PSMN1R0-40YLD, SMD_Packages:LFPAK56_SO8_SOT1023, F.Cu at (110.2, 93.8)
- added Q11: PSMN1R0-40YLD, SMD_Packages:LFPAK56_SO8_SOT1023, F.Cu at (147.6, 64.6)
- added Q12: PSMN1R0-40YLD, SMD_Packages:LFPAK56_SO8_SOT1023, F.Cu at (147.6, 73.6)
- added Q13: PSMN1R0-40YLD, SMD_Packages:LFPAK56_SO8_SOT1023, F.Cu at (123.5, 93.8)
- added Q14: PSMN1R0-40YLD, SMD_Packages:LFPAK56_SO8_SOT1023, F.Cu at (110.2, 133.5)
- added Q15: PSMN1R0-40YLD, SMD_Packages:LFPAK56_SO8_SOT1023, F.Cu at (143.6, 118.4)
- added Q16: PSMN1R0-40YLD, SMD_Packages:LFPAK56_SO8_SOT1023, F.Cu at (156.8, 109.4)
- added Q17: PSMN1R0-40YLD, SMD_Packages:LFPAK56_SO8_SOT1023, F.Cu at (136.7, 127.5)
- added R39: 10, Resistors_SMD:R_0603, F.Cu at (165.9, 75.5)
- added R40: 10, Resistors_SMD:R_0603, F.Cu at (160.0, 82.7)
- added R41: 10k, Resistors_SMD:R_0603, F.Cu at (147.5, 96.0)
- added R42: 10k, Resistors_SMD:R_0603, F.Cu at (150.8, 97.8)
- added R43: 10k, Resistors_SMD:R_0603, F.Cu at (154.9, 92.8)
- added R44: 10k, Resistors_SMD:R_0603, F.Cu at (169.2, 77.6)
- added R45: 10, Resistors_SMD:R_0603, F.Cu at (163.3, 82.7)
- added R46: 10, Resistors_SMD:R_0603, F.Cu at (169.6, 72.6)
- added R47: 10, Resistors_SMD:R_0603, F.Cu at (174.4, 122.4)
- added R48: 10, Resistors_SMD:R_0603, F.Cu at (164.9, 132.4)
- added R49: 10k, Resistors_SMD:R_0603, F.Cu at (157.4, 139.1)
- added R50: 10k, Resistors_SMD:R_0603, F.Cu at (154.1, 139.1)
- added R51: 10k, Resistors_SMD:R_0603, F.Cu at (161.6, 132.4)
- added R52: 10k, Resistors_SMD:R_0603, F.Cu at (165.3, 127.4)
- added R53: 10, Resistors_SMD:R_0603, F.Cu at (158.7, 127.4)
- added R54: 10, Resistors_SMD:R_0603, F.Cu at (158.3, 134.1)
- J19, J20, JP2, U7: moved to B.Cu
- moved R5 225.9 mm to (246.8, 68.6)
- moved R4 202.2 mm to (209.9, 97.2)
- moved R11 202.2 mm to (206.7, 97.2)
- moved R7 202.0 mm to (194.4, 97.2)
- moved D1 201.9 mm to (229.1, 83.0)
- moved J6 201.6 mm to (210.6, 87.7)
- moved J7 200.1 mm to (236.2, 73.7)
- moved D4 198.4 mm to (243.0, 75.4)
- moved D5 193.7 mm to (232.4, 83.0)
- moved J8 191.9 mm to (222.3, 87.7)
- moved J1 190.5 mm to (185.8, 87.7)
- moved J10 190.5 mm to (195.9, 63.2)
- moved J11 190.5 mm to (205.9, 63.2)
- moved J12 190.5 mm to (216.0, 63.2)
- moved J5 190.5 mm to (226.0, 63.4)
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Connections:
- R21 pad 1: Net-(Q2-Pad4) -> Net-(R21-Pad1)
- R21 pad 2: Net-(R21-Pad2) -> Net-(Q2-Pad4)
- R22 pad 1: Net-(Q3-Pad4) -> Net-(C21-Pad2)
- R22 pad 2: Net-(C21-Pad2) -> Net-(Q3-Pad4)
- R27 pad 1: Net-(R27-Pad1) -> Net-(Q4-Pad4)
- R27 pad 2: Net-(Q4-Pad4) -> Net-(R27-Pad2)
- R28 pad 1: Net-(R28-Pad1) -> Net-(Q5-Pad4)
- R28 pad 2: Net-(Q5-Pad4) -> Net-(R28-Pad2)
- R31 pad 1: Net-(Q6-Pad4) -> Net-(R31-Pad1)
- R31 pad 2: Net-(R31-Pad2) -> Net-(Q6-Pad4)
- R32 pad 1: Net-(Q7-Pad4) -> Net-(C28-Pad2)
- R32 pad 2: Net-(C28-Pad2) -> Net-(Q7-Pad4)
- R37 pad 1: Net-(R37-Pad1) -> Net-(Q8-Pad4)
- R37 pad 2: Net-(Q8-Pad4) -> Net-(R37-Pad2)
- R38 pad 1: Net-(R38-Pad1) -> Net-(Q9-Pad4)
- R38 pad 2: Net-(Q9-Pad4) -> Net-(R38-Pad2)
- U4 pad 18: Net-(R28-Pad1) -> Net-(R28-Pad2)
- U4 pad 20: Net-(R27-Pad1) -> Net-(R27-Pad2)
- U4 pad 24: Net-(R21-Pad2) -> Net-(R21-Pad1)
- U6 pad 18: Net-(R38-Pad1) -> Net-(R38-Pad2)
- U6 pad 20: Net-(R37-Pad1) -> Net-(R37-Pad2)
- U6 pad 24: Net-(R31-Pad2) -> Net-(R31-Pad1)
Other:
- board outline removed

Commit message: しんちょく
Parts:
- R25: renamed from R39; moved to B.Cu
- R26: renamed from R40; moved to B.Cu
- moved J23 145.7 mm to (29.0, 152.0), turned to 90 degrees
- moved J16 134.1 mm to (29.0, 97.0)
- moved J22 134.0 mm to (29.0, 144.0), turned to 90 degrees
- moved J18 130.3 mm to (29.0, 81.0)
- moved R23 124.0 mm to (43.0, 73.0)
- moved J21 119.4 mm to (29.0, 136.0), turned to 90 degrees
- moved J17 118.9 mm to (29.0, 89.0)
- moved R26 118.1 mm to (42.0, 79.0), turned to 180 degrees
- moved R21 116.4 mm to (43.0, 71.0), turned to 180 degrees
- moved R25 116.0 mm to (50.0, 79.0), turned to 180 degrees
- moved U5 113.2 mm to (60.0, 100.0), turned to 0 degrees
- moved R22 112.7 mm to (50.0, 71.0), turned to 180 degrees
- moved Q5 111.0 mm to (38.0, 82.0)
- moved J15 107.2 mm to (29.0, 73.0)
- moved Q14 106.9 mm to (56.0, 145.0), turned to 270 degrees
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- renumbered J14 to J13, J13 to J14, J16 to J15, J15 to J16, J20 to J19, J19 to J20, J22 to J21, J21 to J22, Q7 to Q10, Q6 to Q11, Q14 to Q12, Q15 to Q13, Q16 to Q14, Q17 to Q15, Q9 to Q16, Q8 to Q17, Q3 to Q2, Q2 to Q3, Q10 to Q4, Q11 to Q5, Q12 to Q6, Q13 to Q7, Q5 to Q8, Q4 to Q9, R41 to R27, R42 to R28, R43 to R29, R44 to R30, R45 to R31, R46 to R32, R26 to R33, R25 to R34, R28 to R35, R27 to R36, R29 to R37, R30 to R38, R31 to R39, R32 to R40, R33 to R41, R34 to R42, R47 to R43, R48 to R44, R49 to R45, R50 to R46, R51 to R47, R52 to R48, R53 to R49, R54 to R50, R36 to R51, R35 to R52, R38 to R53, R37 to R54
Routing:
- added copper zone on F.Cu, net Net-(Q10-Pad5)
Other:
- board outline added: 50 x 105 mm

Commit message: 進捗セーブ
Parts:
- J15, J16, J17, J18, J21, J22, J23, J24: footprint Mounting_Holes:MountingHole_3mm_Pad_Via -> Mounting_Holes:MountingHole_2.7mm_Pad_Via
- R39, R41, R44, R46: moved to B.Cu
- U7: moved to F.Cu
- moved C30 68.7 mm to (34.8, 119.0)
- moved U7 62.6 mm to (34.7, 124.6)
- moved R44 56.5 mm to (42.4, 131.1), turned to 270 degrees
- moved JP2 50.9 mm to (34.8, 123.5), turned to 270 degrees
- moved R46 50.8 mm to (40.9, 131.1), turned to 270 degrees
- moved R41 50.3 mm to (34.9, 131.1), turned to 270 degrees
- moved R39 45.4 mm to (36.4, 131.1), turned to 270 degrees
- moved C29 39.1 mm to (61.0, 137.7), turned to 90 degrees
- moved C27 37.8 mm to (59.0, 140.0)
- moved C28 3.76 mm to (61.0, 142.2), turned to 270 degrees
- moved Q10 2.37 mm to (49.0, 132.8)
- moved Q12 2.37 mm to (55.0, 132.8)
- moved Q14 2.37 mm to (55.0, 147.2)
- moved Q16 2.37 mm to (49.0, 147.2)
- moved U6 2.00 mm to (67.0, 140.0), turned to 90 degrees
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Routing:
- net GND: track 0.00 -> 60.5 mm, vias 0 -> 36
- net Net-(Q10-Pad5): track 0.00 -> 32.7 mm, vias 0 -> 2
- net Net-(R39-Pad1): track 0.00 -> 9.99 mm, vias 0 -> 1
- net Net-(C27-Pad2): track 0.00 -> 5.05 mm
- net Net-(C29-Pad1): track 0.00 -> 4.81 mm
- net Net-(J20-Pad9): track 0.00 -> 4.50 mm, vias 0 -> 1
- net Net-(C28-Pad1): track 0.00 -> 4.28 mm
- net Net-(Q13-Pad4): track 0.00 -> 4.08 mm, vias 0 -> 1
- net Net-(Q11-Pad4): track 0.00 -> 4.08 mm, vias 0 -> 1
- net +3V3: track 0.00 -> 2.92 mm
- net Net-(Q12-Pad4): track 0.00 -> 1.60 mm, vias 0 -> 1
- net Net-(Q10-Pad4): track 0.00 -> 1.60 mm, vias 0 -> 1
- net Net-(Q15-Pad4): track 0.00 -> 1.46 mm, vias 0 -> 1
- net Net-(Q17-Pad4): track 0.00 -> 1.41 mm, vias 0 -> 1
- net Net-(Q16-Pad4): track 0.00 -> 1.26 mm, vias 0 -> 1
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- added copper zone on B.Cu, net GND
- added copper zone on F.Cu, net GND
- added copper zone on F.Cu, net Net-(C29-Pad2)
- added copper zone on F.Cu, net Net-(J24-Pad1)
- added copper zone on F.Cu, net V_BATT

Commit message: 進捗セーブ
Parts:
- C27, R38, R40, R42, R43, R45, R47, R48, R49, R50, R51, R52, R53, R54: moved to B.Cu
- moved R48 58.1 mm to (38.1, 147.6), turned to 180 degrees
- moved R50 49.1 mm to (40.2, 147.8), turned to 270 degrees
- moved R51 43.3 mm to (49.5, 146.0)
- moved R52 42.2 mm to (43.8, 147.5), turned to 180 degrees
- moved R54 42.2 mm to (45.9, 147.8), turned to 270 degrees
- moved R45 40.3 mm to (54.8, 134.0)
- moved R42 39.4 mm to (48.8, 134.0)
- moved R47 37.2 mm to (55.5, 146.0)
- moved R49 36.2 mm to (53.4, 146.5), turned to 270 degrees
- moved C26 33.9 mm to (69.9, 145.4), turned to 180 degrees
- moved D11 33.0 mm to (65.6, 145.4), turned to 180 degrees
- moved R53 32.8 mm to (47.4, 146.5), turned to 270 degrees
- moved R38 32.2 mm to (62.0, 131.0)
- moved R43 28.4 mm to (56.9, 133.5), turned to 270 degrees
- moved R40 27.4 mm to (50.9, 133.5), turned to 270 degrees
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Connections:
- J14 pad 1: V_BATT -> Net-(J14-Pad1)
- J14 pad 10: GND -> (no net)
- J14 pad 2: (no net) -> V_BATT
- J14 pad 3: (no net) -> GND
- J14 pad 5: (no net) -> +3V3
- J14 pad 8: +3V3 -> (no net)
- J14 pad 9: Net-(J14-Pad9) -> (no net)
- J17 pad 1: Net-(C22-Pad2) -> Net-(J17-Pad1)
- J20 pad 1: V_BATT -> Net-(J20-Pad1)
- J20 pad 10: GND -> (no net)
- J20 pad 2: (no net) -> V_BATT
- J20 pad 3: (no net) -> GND
- J20 pad 5: (no net) -> +3V3
- J20 pad 8: +3V3 -> (no net)
- J20 pad 9: Net-(J20-Pad9) -> (no net)
- J23 pad 1: Net-(C29-Pad2) -> Net-(J23-Pad1)
- Q10 pad 5: Net-(Q10-Pad5) -> Net-(C29-Pad2)
- Q11 pad 1: Net-(Q10-Pad5) -> Net-(C29-Pad2)
- Q11 pad 2: Net-(Q10-Pad5) -> Net-(C29-Pad2)
- Q11 pad 3: Net-(Q10-Pad5) -> Net-(C29-Pad2)
- Q12 pad 5: Net-(Q10-Pad5) -> Net-(C29-Pad2)
- Q13 pad 1: Net-(Q10-Pad5) -> Net-(C29-Pad2)
- Q13 pad 2: Net-(Q10-Pad5) -> Net-(C29-Pad2)
- Q13 pad 3: Net-(Q10-Pad5) -> Net-(C29-Pad2)
- Q14 pad 5: Net-(C29-Pad2) -> Net-(J23-Pad1)
- Q15 pad 1: Net-(C29-Pad2) -> Net-(J23-Pad1)
- Q15 pad 2: Net-(C29-Pad2) -> Net-(J23-Pad1)
- Q15 pad 3: Net-(C29-Pad2) -> Net-(J23-Pad1)
- Q16 pad 5: Net-(C29-Pad2) -> Net-(J23-Pad1)
- Q17 pad 1: Net-(C29-Pad2) -> Net-(J23-Pad1)
- Q17 pad 2: Net-(C29-Pad2) -> Net-(J23-Pad1)
- Q17 pad 3: Net-(C29-Pad2) -> Net-(J23-Pad1)
- Q2 pad 5: Net-(Q2-Pad5) -> Net-(C22-Pad2)
- Q3 pad 1: Net-(Q2-Pad5) -> Net-(C22-Pad2)
- Q3 pad 2: Net-(Q2-Pad5) -> Net-(C22-Pad2)
- Q3 pad 3: Net-(Q2-Pad5) -> Net-(C22-Pad2)
- Q4 pad 5: Net-(Q2-Pad5) -> Net-(C22-Pad2)
- Q5 pad 1: Net-(Q2-Pad5) -> Net-(C22-Pad2)
- Q5 pad 2: Net-(Q2-Pad5) -> Net-(C22-Pad2)
- Q5 pad 3: Net-(Q2-Pad5) -> Net-(C22-Pad2)
- Q6 pad 5: Net-(C22-Pad2) -> Net-(J17-Pad1)
- Q7 pad 1: Net-(C22-Pad2) -> Net-(J17-Pad1)
- Q7 pad 2: Net-(C22-Pad2) -> Net-(J17-Pad1)
- Q7 pad 3: Net-(C22-Pad2) -> Net-(J17-Pad1)
- Q8 pad 5: Net-(C22-Pad2) -> Net-(J17-Pad1)
- Q9 pad 1: Net-(C22-Pad2) -> Net-(J17-Pad1)
- Q9 pad 2: Net-(C22-Pad2) -> Net-(J17-Pad1)
- Q9 pad 3: Net-(C22-Pad2) -> Net-(J17-Pad1)
- R22 pad 1: Net-(C21-Pad2) -> Net-(R22-Pad1)
- R23 pad 1: Net-(Q2-Pad5) -> Net-(C22-Pad2)
- R25 pad 1: Net-(C21-Pad2) -> Net-(R22-Pad1)
- R28 pad 1: Net-(Q2-Pad5) -> Net-(C22-Pad2)
- R30 pad 2: Net-(C22-Pad2) -> Net-(J17-Pad1)
- R31 pad 2: Net-(R31-Pad2) -> Net-(C21-Pad2)
- R34 pad 2: Net-(C22-Pad2) -> Net-(J17-Pad1)
- R35 pad 2: Net-(R31-Pad2) -> Net-(C21-Pad2)
- R40 pad 1: Net-(C28-Pad2) -> Net-(R40-Pad1)
- R41 pad 1: Net-(Q10-Pad5) -> Net-(C29-Pad2)
- R43 pad 1: Net-(C28-Pad2) -> Net-(R40-Pad1)
- R46 pad 1: Net-(Q10-Pad5) -> Net-(C29-Pad2)
- R48 pad 2: Net-(C29-Pad2) -> Net-(J23-Pad1)
- R49 pad 2: Net-(R49-Pad2) -> Net-(C28-Pad2)
- R52 pad 2: Net-(C29-Pad2) -> Net-(J23-Pad1)
- R53 pad 2: Net-(R49-Pad2) -> Net-(C28-Pad2)
- U4 pad 1: Net-(Q2-Pad5) -> Net-(J17-Pad1)
- U4 pad 18: Net-(R31-Pad2) -> Net-(R22-Pad1)
- U4 pad 20: Net-(R32-Pad2) -> Net-(R21-Pad1)
- U4 pad 24: Net-(R21-Pad1) -> Net-(R32-Pad2)
- U5 pad 3: Net-(Q2-Pad5) -> Net-(C22-Pad2)
- U5 pad 4: Net-(Q2-Pad5) -> Net-(C22-Pad2)
- U5 pad 7: Net-(J14-Pad9) -> Net-(J14-Pad1)
- U6 pad 1: Net-(Q10-Pad5) -> Net-(J23-Pad1)
- U6 pad 18: Net-(R49-Pad2) -> Net-(R40-Pad1)
- U6 pad 20: Net-(R50-Pad2) -> Net-(R39-Pad1)
- U6 pad 24: Net-(R39-Pad1) -> Net-(R50-Pad2)
- U7 pad 3: Net-(Q10-Pad5) -> Net-(C29-Pad2)
- U7 pad 4: Net-(Q10-Pad5) -> Net-(C29-Pad2)
- U7 pad 7: Net-(J20-Pad9) -> Net-(J20-Pad1)
Routing:
- net V_BATT: track 0.00 -> 69.0 mm
- net GND: track 60.5 -> 117.7 mm, vias 36 -> 37
- net Net-(C29-Pad2): track 0.00 -> 42.7 mm, vias 0 -> 2
- net +3V3: track 2.92 -> 35.8 mm, vias 0 -> 2
- net Net-(Q10-Pad5): track 32.7 -> 0.00 mm, vias 2 -> 0
- net Net-(J23-Pad1): track 0.00 -> 24.1 mm, vias 0 -> 2
- net Net-(J20-Pad1): track 0.00 -> 23.1 mm, vias 0 -> 1
- net Net-(R39-Pad1): track 9.99 -> 31.2 mm
- net Net-(R50-Pad2): track 0.00 -> 21.2 mm, vias 0 -> 1
- net Net-(R40-Pad1): track 0.00 -> 15.6 mm, vias 0 -> 1
- net Net-(C28-Pad2): track 0.00 -> 11.7 mm
- net Net-(J24-Pad1): track 0.00 -> 6.28 mm
- net Net-(JP2-Pad2): track 0.00 -> 5.15 mm, vias 0 -> 1
- net Net-(J20-Pad9): track 4.50 -> 0.00 mm, vias 1 -> 0
- net Net-(Q16-Pad4): track 1.26 -> 4.33 mm
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- added copper zone on F.Cu, net Net-(J23-Pad1)
- removed copper zone on F.Cu, net Net-(Q10-Pad5)
Other:
- outline, holes or cut-outs redrawn

Commit message: 一度全部配線はできた，きれいにする必要あり
Parts:
- removed J13, J19: CONN_01X10, Pin_Headers:Pin_Header_Straight_1x10_Pitch2.00mm_SMD_Pin1Left
- R37: moved to B.Cu
- moved R37 7.29 mm to (61.7, 126.5)
- moved C26 4.21 mm to (65.9, 144.1)
- moved J20 4.12 mm to (60.0, 122.0)
- moved D11 4.10 mm to (62.7, 148.3)
- moved R38 4.10 mm to (66.1, 131.1), turned to 90 degrees
- moved C24 2.55 mm to (66.8, 136.6), turned to 180 degrees
- moved C29 2.39 mm to (59.0, 139.0), turned to 180 degrees
- moved C28 2.36 mm to (59.0, 141.0), turned to 180 degrees
- moved C25 1.00 mm to (66.6, 148.3)
- moved U6 0.80 mm to (64.6, 140.0)
Connections:
- J14 pad 10: (no net) -> Net-(J14-Pad10)
- J14 pad 4: (no net) -> Net-(J14-Pad4)
- J14 pad 6: (no net) -> Net-(J14-Pad6)
- J14 pad 7: (no net) -> Net-(J14-Pad7)
- J14 pad 8: (no net) -> Net-(J14-Pad8)
- J14 pad 9: (no net) -> Net-(J14-Pad9)
- J17 pad 1: Net-(J17-Pad1) -> Net-(C21-Pad2)
- J20 pad 10: (no net) -> Net-(J20-Pad10)
- J20 pad 4: (no net) -> Net-(J20-Pad4)
- J20 pad 6: (no net) -> Net-(J20-Pad6)
- J20 pad 7: (no net) -> Net-(J20-Pad7)
- J20 pad 8: (no net) -> Net-(J20-Pad8)
- J20 pad 9: (no net) -> Net-(J20-Pad9)
- J23 pad 1: Net-(J23-Pad1) -> Net-(C28-Pad2)
- Q14 pad 5: Net-(J23-Pad1) -> Net-(C28-Pad2)
- Q15 pad 1: Net-(J23-Pad1) -> Net-(C28-Pad2)
- Q15 pad 2: Net-(J23-Pad1) -> Net-(C28-Pad2)
- Q15 pad 3: Net-(J23-Pad1) -> Net-(C28-Pad2)
- Q16 pad 5: Net-(J23-Pad1) -> Net-(C28-Pad2)
- Q17 pad 1: Net-(J23-Pad1) -> Net-(C28-Pad2)
- Q17 pad 2: Net-(J23-Pad1) -> Net-(C28-Pad2)
- Q17 pad 3: Net-(J23-Pad1) -> Net-(C28-Pad2)
- Q6 pad 5: Net-(J17-Pad1) -> Net-(C21-Pad2)
- Q7 pad 1: Net-(J17-Pad1) -> Net-(C21-Pad2)
- Q7 pad 2: Net-(J17-Pad1) -> Net-(C21-Pad2)
- Q7 pad 3: Net-(J17-Pad1) -> Net-(C21-Pad2)
- Q8 pad 5: Net-(J17-Pad1) -> Net-(C21-Pad2)
- Q9 pad 1: Net-(J17-Pad1) -> Net-(C21-Pad2)
- Q9 pad 2: Net-(J17-Pad1) -> Net-(C21-Pad2)
- Q9 pad 3: Net-(J17-Pad1) -> Net-(C21-Pad2)
- R19 pad 2: Net-(J13-Pad7) -> Net-(J14-Pad6)
- R30 pad 2: Net-(J17-Pad1) -> Net-(C21-Pad2)
- R31 pad 2: Net-(C21-Pad2) -> Net-(R31-Pad2)
- R34 pad 2: Net-(J17-Pad1) -> Net-(C21-Pad2)
- R35 pad 2: Net-(C21-Pad2) -> Net-(R31-Pad2)
- R37 pad 2: Net-(J19-Pad7) -> Net-(J20-Pad6)
- R48 pad 2: Net-(J23-Pad1) -> Net-(C28-Pad2)
- R49 pad 2: Net-(C28-Pad2) -> Net-(R49-Pad2)
- R52 pad 2: Net-(J23-Pad1) -> Net-(C28-Pad2)
- R53 pad 2: Net-(C28-Pad2) -> Net-(R49-Pad2)
- U4 pad 1: Net-(J17-Pad1) -> Net-(C21-Pad2)
- U4 pad 10: Net-(J13-Pad3) -> Net-(J14-Pad8)
- U4 pad 11: Net-(J13-Pad2) -> Net-(J14-Pad7)
- U4 pad 15: Net-(J13-Pad7) -> Net-(J14-Pad6)
- U4 pad 16: Net-(J13-Pad6) -> Net-(J14-Pad4)
- U4 pad 2: Net-(C21-Pad2) -> Net-(R31-Pad2)
- U4 pad 8: Net-(J13-Pad5) -> Net-(J14-Pad10)
- U4 pad 9: Net-(J13-Pad4) -> Net-(J14-Pad9)
- U6 pad 1: Net-(J23-Pad1) -> Net-(C28-Pad2)
- U6 pad 10: Net-(J19-Pad3) -> Net-(J20-Pad8)
- U6 pad 11: Net-(J19-Pad2) -> Net-(J20-Pad7)
- U6 pad 15: Net-(J19-Pad7) -> Net-(J20-Pad6)
- U6 pad 16: Net-(J19-Pad6) -> Net-(J20-Pad4)
- U6 pad 2: Net-(C28-Pad2) -> Net-(R49-Pad2)
- U6 pad 8: Net-(J19-Pad5) -> Net-(J20-Pad10)
- U6 pad 9: Net-(J19-Pad4) -> Net-(J20-Pad9)
Routing:
- net V_BATT: track 69.0 -> 117.3 mm, vias 0 -> 1
- net GND: track 117.7 -> 153.6 mm, vias 37 -> 47
- net Net-(C28-Pad2): track 11.7 -> 37.5 mm, vias 0 -> 2
- net Net-(J20-Pad9): track 0.00 -> 24.4 mm, vias 0 -> 1
- net +3V3: track 35.8 -> 60.0 mm, vias 2 -> 3
- net Net-(J23-Pad1): track 24.1 -> 0.00 mm, vias 2 -> 0
- net Net-(J20-Pad7): track 0.00 -> 24.0 mm, vias 0 -> 1
- net Net-(J20-Pad10): track 0.00 -> 20.3 mm, vias 0 -> 1
- net Net-(J20-Pad8): track 0.00 -> 19.2 mm, vias 0 -> 1
- net Net-(R49-Pad2): track 0.00 -> 19.1 mm, vias 0 -> 1
- net Net-(J20-Pad6): track 0.00 -> 19.0 mm, vias 0 -> 1
- net Net-(J20-Pad4): track 0.00 -> 17.5 mm, vias 0 -> 1
- net Net-(R38-Pad2): track 0.00 -> 9.01 mm, vias 0 -> 1
- net Net-(C25-Pad1): track 0.00 -> 7.75 mm
- net Net-(R50-Pad2): track 21.2 -> 28.0 mm
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- added copper zone on F.Cu, net Net-(C28-Pad2)
- removed copper zone on F.Cu, net Net-(J23-Pad1)
Other:
- board size 50 x 105 mm -> 50 x 94 mm

Commit message: しんちょくセーブ
Parts:
- removed JP1, JP2: Jumper_NC_Dual, Connect:GS3
- added C31: C, Capacitors_SMD:C_0603, F.Cu at (81.9, 75.5)
- added C32: C, Capacitors_SMD:C_0603, B.Cu at (40.7, 125.7)
- U1: moved to B.Cu
- U5: value ACS722 -> ACS711; footprint SMD_Packages:SOIC-8-N -> Housings_DFN_QFN:QFN-12_3x3mm_Pitch0.5mm_With_Fused_Sensed_Current_Loop; moved to F.Cu
- U7: value ACS722 -> ACS711; footprint SMD_Packages:SOIC-8-N -> Housings_DFN_QFN:QFN-12_3x3mm_Pitch0.5mm_With_Fused_Sensed_Current_Loop
- moved U1 121.7 mm to (108.0, 109.0), turned to 90 degrees
- moved J10 115.1 mm to (100.0, 127.0), turned to 90 degrees
- moved J9 91.2 mm to (100.0, 94.0), turned to 90 degrees
- moved U5 55.8 mm to (37.0, 49.2)
- moved C17 37.4 mm to (50.6, 53.2)
- moved R33 37.4 mm to (54.4, 65.4)
- moved R34 37.4 mm to (57.4, 55.4)
- moved C19 37.4 mm to (56.9, 50.3)
- moved C21 37.4 mm to (57.7, 45.3)
- moved R24 37.4 mm to (57.0, 60.3)
- moved R30 37.4 mm to (53.7, 60.3)
- moved R32 37.4 mm to (54.1, 55.3)
- moved R20 36.8 mm to (75.7, 59.4)
- moved C20 36.8 mm to (71.7, 57.4)
- moved R28 36.8 mm to (74.9, 64.4)
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Connections:
- U5 pad 6: Net-(JP1-Pad2) -> (no net)
- U7 pad 6: Net-(JP2-Pad2) -> (no net)
Routing:
- net V_BATT: track 117.3 -> 108.6 mm
- net Net-(J20-Pad9): track 24.4 -> 17.9 mm
- net Net-(J20-Pad10): track 20.3 -> 13.9 mm
- net Net-(J20-Pad7): track 24.0 -> 17.6 mm
- net Net-(JP2-Pad2): track 5.15 -> 0.00 mm, vias 1 -> 0
- net Net-(J20-Pad8): track 19.2 -> 14.1 mm
- net Net-(J20-Pad6): track 19.0 -> 14.5 mm
- net Net-(J20-Pad4): track 17.5 -> 13.3 mm
- net +3V3: track 60.0 -> 56.2 mm, vias 3 -> 2
- net Net-(R38-Pad2): track 9.01 -> 6.56 mm
- net GND: track 153.6 -> 151.6 mm, vias 47 -> 50
- net Net-(R49-Pad2): track 19.1 -> 21.0 mm
- net Net-(C32-Pad1): track 18.5 -> 20.2 mm
- net Net-(C28-Pad2): track 37.5 -> 38.9 mm
Other:
- board size 50 x 94 mm -> 95 x 69 mm
