File: nmkgmmd_v10_brd.kicad_pcb (KiCad board)
At the start: 2 copper layers, 95 x 69 mm, 150 parts, among them J1 CONN_01X05, J10 CONN_01X10, J11 CONN_01X10, J12 CONN_01X10, J14 CONN_01X10, J15 CONN_01X01, J16 CONN_01X01, J17 CONN_01X01, J18 CONN_01X01, J2 CONN_01X03, J20 CONN_01X10, J21 CONN_01X01, J22 CONN_01X01, J23 CONN_01X01, J24 CONN_01X01, J3 CONN_01X03, J4 CONN_01X04, J5 CONN_01X04, J6 CONN_01X04, J7 CONN_01X03, J8 CONN_01X03, J9 CONN_01X10, Q1 BSS138PS, Q10 PSMN1R0-40YLD, Q11 PSMN1R0-40YLD, Q12 PSMN1R0-40YLD, Q13 PSMN1R0-40YLD, Q14 PSMN1R0-40YLD, Q15 PSMN1R0-40YLD, Q16 PSMN1R0-40YLD, Q17 PSMN1R0-40YLD, Q2 PSMN1R0-40YLD, Q3 PSMN1R0-40YLD, Q4 PSMN1R0-40YLD, Q5 PSMN1R0-40YLD, Q6 PSMN1R0-40YLD, Q7 PSMN1R0-40YLD, Q8 PSMN1R0-40YLD, Q9 PSMN1R0-40YLD, SW1 SKRPACE010, SW2 SW_DPDT_x2, U1 STM32F303CCTx, U2 MCP16301, U3 MCP16301, U4 A4957, U5 ACS711, U6 A4957, U7 ACS711, Y1 Crystal

Commit message: セーブ
Parts:
- removed J11, J12: CONN_01X10, Pin_Headers:Pin_Header_Straight_1x10_Pitch2.00mm
- C2, C3, D3, D4, D5, L2, SW1, SW2, Y1: moved to B.Cu
- J10, J9: footprint Pin_Headers:Pin_Header_Straight_1x10_Pitch2.00mm -> Pin_Headers:Pin_Header_Straight_1x10_Pitch2.00mm_SMD_Pin1Right
- moved L1 158.7 mm to (102.3, 140.9), turned to 180 degrees
- moved D4 151.9 mm to (96.7, 116.5), turned to 270 degrees
- moved L2 150.5 mm to (96.6, 110.1), turned to 270 degrees
- moved SW1 150.2 mm to (92.1, 85.7)
- moved J5 148.8 mm to (105.4, 150.5), turned to 90 degrees
- moved R12 144.3 mm to (116.5, 139.1), turned to 90 degrees
- moved Q1 142.1 mm to (124.1, 134.6), turned to 90 degrees
- moved C8 141.7 mm to (116.6, 142.5), turned to 90 degrees
- moved D5 141.2 mm to (95.2, 116.5), turned to 270 degrees
- moved C4 139.3 mm to (116.6, 146.0), turned to 90 degrees
- moved R5 134.5 mm to (129.6, 134.7), turned to 90 degrees
- moved C7 128.6 mm to (123.6, 148.9), turned to 90 degrees
- moved C6 126.5 mm to (123.4, 152.6), turned to 90 degrees
- moved C2 123.6 mm to (97.6, 106.3), turned to 180 degrees
- moved C3 123.6 mm to (97.6, 101.1), turned to 180 degrees
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Connections:
- J10 pad 1: +3V3 -> /MCU/A2_IN12
- J10 pad 10: GND -> /MCU/T8_CH2N
- J10 pad 2: /MCU/T8_CH1 -> V_BATT
- J10 pad 3: /MCU/T8_CH1N -> GND
- J10 pad 4: /MCU/T8_CH2 -> /MCU/RESET2
- J10 pad 5: /MCU/T8_CH2N -> +3V3
- J10 pad 6: /MCU/RESET2 -> /MCU/FAULT2
- J10 pad 7: /MCU/FAULT2 -> /MCU/T8_CH1
- J10 pad 8: (no net) -> /MCU/T8_CH1N
- J10 pad 9: (no net) -> /MCU/T8_CH2
- J9 pad 1: +3V3 -> /MCU/A3_IN1
- J9 pad 10: GND -> /MCU/T1_CH2N
- J9 pad 2: /MCU/T1_CH1 -> V_BATT
- J9 pad 3: /MCU/T1_CH1N -> GND
- J9 pad 4: /MCU/T1_CH2 -> /MCU/RESET1
- J9 pad 5: /MCU/T1_CH2N -> +3V3
- J9 pad 6: /MCU/RESET1 -> /MCU/FAULT1
- J9 pad 7: /MCU/FAULT1 -> /MCU/T1_CH1
- J9 pad 8: (no net) -> /MCU/T1_CH1N
- J9 pad 9: (no net) -> /MCU/T1_CH2
Routing:
- net /MCU/T1_CH1N: track 0.00 -> 17.5 mm, vias 0 -> 1
- net Net-(C3-Pad2): track 0.00 -> 7.70 mm
- net Net-(C2-Pad2): track 0.00 -> 7.09 mm
- added copper zone on F.Cu, net Net-(J18-Pad1)
Other:
- board size 95 x 69 mm -> 85 x 69 mm
