File: nmkgmmd_v10_brd.sch (KiCad schematic (older format))
At the start: 28 parts, among them J1 CONN_01X05, J10 CONN_01X10, J2 CONN_01X03, J3 CONN_01X03, J4 CONN_01X04, J5 CONN_01X04, J6 CONN_01X04, J7 CONN_01X03, J8 CONN_01X03, J9 CONN_01X10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

Commit message: ネットリスト更新，進捗
Connections:
- net MCU/A2_IN12: now also J9.1 (P1); no longer J10.1 (P1)
- net MCU/A3_IN1: now also J10.1 (P1); no longer J9.1 (P1)
Changed lines of the file:
@@
 F21 "T3_CH1" I L 5750 3650 60
 F22 "T2_CH2" I L 5750 3350 60
-F23 "A2_IN12" I R 6750 4650 60
-F24 "A3_IN1" I R 6750 3600 60
+F23 "A2_IN12" I R 6750 3600 60
+F24 "A3_IN1" I R 6750 4650 60
 F25 "T8_CH2N" O R 6750 4200 60
 F26 "T1_CH1N" O R 6750 2900 60
@@
 	5750 4150 4550 4150
 Wire Wire Line
-	4550 4850 4550 4150
+	4550 4150 4550 4850
 Wire Wire Line
 	4400 4050 5750 4050
@@
 Connection ~ 3250 4050
 Wire Wire Line
-	3950 4850 4550 4850
+	4550 4850 3950 4850
 Wire Wire Line
 	4300 4800 4300 4850
@@
 	7950 2250 7950 3600
 Wire Wire Line
-	7950 3600 6750 3600
-Wire Wire Line
 	8450 4000 7150 4000
 Wire Wire Line
 	7150 4000 7150 4650
-Wire Wire Line
-	7150 4650 6750 4650
 Wire Wire Line
 	8500 2550 8050 2550
@@
 Wire Wire Line
 	5150 2900 5150 3350
+Wire Wire Line
+	7950 3600 6750 3600
+Wire Wire Line
+	7150 4650 6750 4650
 $EndSCHEMATC

Commit message: 進捗
Parts:
- removed Q1: BSS138PS, TO_SOT_Packages_SMD:SOT-363_SC-70-6, symbol BSS138PS
- added Q1, Q18: BSS138, TO_SOT_Packages_SMD:SOT-23, symbol BSS138
Connections:
- net +3V3: now also Q1.1 (G), Q18.1 (G)
- net MCU/T15_CH2: now also R6.2, Q18.2 (S); no longer R5.2
- net MCU/T4_CH2: now also R5.2, Q1.2 (S); no longer R6.2
- net at J2.3 (P3), R4.2: now also Q1.3 (D)
- net at J3.3 (P3), R3.2: now also Q18.3 (D)
Other:
- moved on the sheet: J2, J3, R3, R4, R5, R6
Changed lines of the file:
@@
 F11 "T1_CH2N" O R 6750 3150 60
 F12 "T2_CH1" I L 5750 3250 60
-F13 "T15_CH2" I L 5750 4050 60
+F13 "T15_CH2" I L 5750 4150 60
 F14 "FAULT1" I R 6750 3450 60
 F15 "FAULT2" I R 6750 4500 60
 F16 "LED0" O L 5750 4650 60
 F17 "T8_CH2" O R 6750 4100 60
-F18 "T4_CH2" I L 5750 4150 60
+F18 "T4_CH2" I L 5750 4050 60
 F19 "T8_CH1" O R 6750 3850 60
 F20 "T3_CH2" I L 5750 3750 60
@@
 L CONN_01X03 J2
 U 1 1 58B81CD5
-P 2550 4350
-F 0 "J2" H 2550 4550 50  0000 C CNN
-F 1 "CONN_01X03" V 2650 4350 50  0000 C CNN
-F 2 "Connectors_JST:JST_ZH_S03B-ZR_03x1.50mm_Angled" H 2550 4350 50  0001 C CNN
-F 3 "" H 2550 4350 50  0001 C CNN
-	1    2550 4350
+P 2850 4350
+F 0 "J2" H 2850 4550 50  0000 C CNN
+F 1 "CONN_01X03" V 2950 4350 50  0000 C CNN
+F 2 "Connectors_JST:JST_ZH_S03B-ZR_03x1.50mm_Angled" H 2850 4350 50  0001 C CNN
+F 3 "" H 2850 4350 50  0001 C CNN
+	1    2850 4350
 	-1   0    0    -1
 $EndComp
@@
 L CONN_01X03 J3
 U 1 1 58B83011
-P 2550 4850
-F 0 "J3" H 2550 5050 50  0000 C CNN
-F 1 "CONN_01X03" V 2650 4850 50  0000 C CNN
-F 2 "Connectors_JST:JST_ZH_S03B-ZR_03x1.50mm_Angled" H 2550 4850 50  0001 C CNN
-F 3 "" H 2550 4850 50  0001 C CNN
-	1    2550 4850
+P 2850 5100
+F 0 "J3" H 2850 5300 50  0000 C CNN
+F 1 "CONN_01X03" V 2950 5100 50  0000 C CNN
+F 2 "Connectors_JST:JST_ZH_S03B-ZR_03x1.50mm_Angled" H 2850 5100 50  0001 C CNN
+F 3 "" H 2850 5100 50  0001 C CNN
+	1    2850 5100
 	-1   0    0    -1
 $EndComp
@@
 L GND #PWR010
 U 1 1 58B8969C
-P 2850 5000
-F 0 "#PWR010" H 2850 4750 50  0001 C CNN
-F 1 "GND" H 2850 4850 50  0000 C CNN
-F 2 "" H 2850 5000 50  0001 C CNN
-F 3 "" H 2850 5000 50  0001 C CNN
-	1    2850 5000
+P 3100 5300
+F 0 "#PWR010" H 3100 5050 50  0001 C CNN
+F 1 "GND" H 3100 5150 50  0000 C CNN
+F 2 "" H 3100 5300 50  0001 C CNN
+F 3 "" H 3100 5300 50  0001 C CNN
+	1    3100 5300
 	1    0    0    -1
 $EndComp
@@
 L +5V #PWR011
 U 1 1 58B8A4F6
-P 2950 4000
-F 0 "#PWR011" H 2950 3850 50  0001 C CNN
-F 1 "+5V" H 2950 4140 50  0000 C CNN
-F 2 "" H 2950 4000 50  0001 C CNN
-F 3 "" H 2950 4000 50  0001 C CNN
-	1    2950 4000
-	1    0    0    -1
-$EndComp
-$Comp
-L BSS138PS Q1
-U 1 1 58BAFB50
-P 3700 4550
-F 0 "Q1" H 3900 5000 50  0000 L CNN
-F 1 "BSS138PS" H 3450 5000 50  0000 L CNN
-F 2 "TO_SOT_Packages_SMD:SOT-363_SC-70-6" V 3625 4950 50  0001 L CIN
-F 3 "" V 3700 4750 50  0000 L CNN
-	1    3700 4550
-	-1   0    0    1
+P 3200 4150
+F 0 "#PWR011" H 3200 4000 50  0001 C CNN
+F 1 "+5V" H 3200 4290 50  0000 C CNN
+F 2 "" H 3200 4150 50  0001 C CNN
+F 3 "" H 3200 4150 50  0001 C CNN
+	1    3200 4150
+	1    0    0    -1
 $EndComp
 $Comp
 L +3V3 #PWR012
 U 1 1 58BB4BA3
-P 4050 4000
-F 0 "#PWR012" H 4050 3850 50  0001 C CNN
-F 1 "+3V3" H 4050 4140 50  0000 C CNN
-F 2 "" H 4050 4000 50  0001 C CNN
-F 3 "" H 4050 4000 50  0001 C CNN
-	1    4050 4000
+P 3950 4150
+F 0 "#PWR012" H 3950 4000 50  0001 C CNN
+F 1 "+3V3" H 3950 4290 50  0000 C CNN
+F 2 "" H 3950 4150 50  0001 C CNN
+F 3 "" H 3950 4150 50  0001 C CNN
+	1    3950 4150
 	1    0    0    -1
 $EndComp
@@
 L R R3
 U 1 1 58BBCAAF
-P 3250 4650
-F 0 "R3" V 3330 4650 50  0000 C CNN
-F 1 "10k" V 3250 4650 50  0000 C CNN
-F 2 "Resistors_SMD:R_0603" V 3180 4650 50  0001 C CNN
-F 3 "" H 3250 4650 50  0001 C CNN
-	1    3250 4650
+P 3300 4650
+F 0 "R3" V 3380 4650 50  0000 C CNN
+F 1 "10k" V 3300 4650 50  0000 C CNN
+F 2 "Resistors_SMD:R_0603" V 3230 4650 50  0001 C CNN
+F 3 "" H 3300 4650 50  0001 C CNN
+	1    3300 4650
 	1    0    0    -1
 $EndComp
@@
 L R R4
 U 1 1 58BBCC08
-P 3400 4250
-F 0 "R4" V 3480 4250 50  0000 C CNN
-F 1 "10k" V 3400 4250 50  0000 C CNN
-F 2 "Resistors_SMD:R_0603" V 3330 4250 50  0001 C CNN
-F 3 "" H 3400 4250 50  0001 C CNN
-	1    3400 4250
+P 3400 4300
+F 0 "R4" V 3480 4300 50  0000 C CNN
+F 1 "10k" V 3400 4300 50  0000 C CNN
+F 2 "Resistors_SMD:R_0603" V 3330 4300 50  0001 C CNN
+F 3 "" H 3400 4300 50  0001 C CNN
+	1    3400 4300
 	1    0    0    -1
 $EndComp
@@
 L R R5
 U 1 1 58BBFB14
-P 4150 4250
-F 0 "R5" V 4230 4250 50  0000 C CNN
-F 1 "10k" V 4150 4250 50  0000 C CNN
-F 2 "Resistors_SMD:R_0603" V 4080 4250 50  0001 C CNN
-F 3 "" H 4150 4250 50  0001 C CNN
-	1    4150 4250
+P 4050 4300
+F 0 "R5" V 4130 4300 50  0000 C CNN
+F 1 "10k" V 4050 4300 50  0000 C CNN
+F 2 "Resistors_SMD:R_0603" V 3980 4300 50  0001 C CNN
+F 3 "" H 4050 4300 50  0001 C CNN
+	1    4050 4300
 	1    0    0    -1
 $EndComp
@@
 L R R6
 U 1 1 58BBFC2A
-P 4300 4650
-F 0 "R6" V 4380 4650 50  0000 C CNN
-F 1 "10k" V 4300 4650 50  0000 C CNN
-F 2 "Resistors_SMD:R_0603" V 4230 4650 50  0001 C CNN
-F 3 "" H 4300 4650 50  0001 C CNN
-	1    4300 4650
+P 4200 4650
+F 0 "R6" V 4280 4650 50  0000 C CNN
+F 1 "10k" V 4200 4650 50  0000 C CNN
+F 2 "Resistors_SMD:R_0603" V 4130 4650 50  0001 C CNN
+F 3 "" H 4200 4650 50  0001 C CNN
+	1    4200 4650
 	1    0    0    -1
 $EndComp
@@
 Text Notes 3850 2300 0    60   ~ 0
 External Analog 2
-Text Notes 1750 4400 0    60   ~ 0
+Text Notes 2100 4400 0    60   ~ 0
 PWM Input 1
-Text Notes 1750 4900 0    60   ~ 0
+Text Notes 2100 5150 0    60   ~ 0
 PWM Input 2
 Text Notes 3750 5650 0    60   ~ 0
@@
 	5750 4150 4550 4150
 Wire Wire Line
-	4550 4150 4550 4850
+	4550 4150 4550 5200
 Wire Wire Line
 	4400 4050 5750 4050
 Wire Wire Line
-	2750 4250 2850 4250
-Wire Wire Line
-	2850 4250 2850 5000
-Wire Wire Line
-	2950 4000 2950 4850
-Wire Wire Line
-	2950 4350 2750 4350
-Connection ~ 2950 4350
+	3050 4250 3100 4250
+Wire Wire Line
+	3100 4250 3100 5300
+Wire Wire Line
+	3200 4150 3400 4150
+Wire Wire Line
+	3200 4150 3200 5100
+Wire Wire Line
+	3200 4350 3050 4350
+Connection ~ 3200 4350
 Wire Wire Line
 	4850 3750 5750 3750
@@
 	5450 2800 5750 2800
 Wire Wire Line
-	4050 4250 3950 4250
-Wire Wire Line
-	4050 4000 4050 4650
-Wire Wire Line
-	4050 4650 3950 4650
-Connection ~ 4050 4250
-Wire Wire Line
-	3250 4950 2750 4950
-Wire Wire Line
-	3250 4800 3250 4950
-Wire Wire Line
-	3250 4850 3450 4850
-Wire Wire Line
-	2750 4450 3450 4450
-Connection ~ 3250 4850
-Wire Wire Line
-	3250 4050 3250 4500
-Wire Wire Line
-	2950 4050 3400 4050
-Wire Wire Line
-	3400 4050 3400 4100
-Connection ~ 2950 4050
-Connection ~ 3250 4050
-Wire Wire Line
-	4550 4850 3950 4850
-Wire Wire Line
-	4300 4800 4300 4850
-Connection ~ 4300 4850
-Wire Wire Line
-	3950 4450 4400 4450
+	3700 4150 4200 4150
+Wire Wire Line
+	3950 4150 3950 4900
+Wire Wire Line
+	3050 5200 3500 5200
+Wire Wire Line
+	3300 4800 3300 5200
+Wire Wire Line
+	3050 4450 3500 4450
+Wire Wire Line
+	3300 4150 3300 4500
+Connection ~ 3200 4150
+Connection ~ 3300 4150
+Wire Wire Line
+	3900 4450 4400 4450
 Wire Wire Line
 	4400 4450 4400 4050
 Wire Wire Line
-	4150 4400 4150 4450
-Connection ~ 4150 4450
-Wire Wire Line
-	4300 4050 4300 4500
-Wire Wire Line
-	4050 4050 4300 4050
-Wire Wire Line
-	4150 4050 4150 4100
-Connection ~ 4050 4050
-Connection ~ 4150 4050
+	4050 4450 4050 4450
+Connection ~ 4050 4450
+Wire Wire Line
+	4200 4150 4200 4500
+Wire Wire Line
+	4050 4150 4050 4150
+Connection ~ 3950 4150
+Connection ~ 4050 4150
 Wire Wire Line
 	2600 2300 2650 2300
@@
 	7550 3850 6750 3850
 Wire Wire Line
-	3400 4400 3400 4450
+	3400 4450 3400 4450
 Connection ~ 3400 4450
 Wire Wire Line
-	2950 4850 2750 4850
-Wire Wire Line
-	2750 4750 2850 4750
-Connection ~ 2850 4750
+	3200 5100 3050 5100
+Wire Wire Line
+	3050 5000 3100 5000
+Connection ~ 3100 5000
 Wire Wire Line
 	4850 3400 4500 3400
@@
 Wire Wire Line
 	7150 4650 6750 4650
+$Comp
+L BSS138 Q1
+U 1 1 58C02AE0
+P 3700 4350
+F 0 "Q1" H 3900 4425 50  0000 L CNN
+F 1 "BSS138" H 3900 4350 50  0000 L CNN
+F 2 "TO_SOT_Packages_SMD:SOT-23" H 3900 4275 50  0001 L CIN
+F 3 "" H 3700 4350 50  0001 L CNN
+	1    3700 4350
+	0    -1   1    0
+$EndComp
+$Comp
+L BSS138 Q18
+U 1 1 58C02EF9
+P 3700 5100
+F 0 "Q18" H 3900 5175 50  0000 L CNN
+F 1 "BSS138" H 3900 5100 50  0000 L CNN
+F 2 "TO_SOT_Packages_SMD:SOT-23" H 3900 5025 50  0001 L CIN
+F 3 "" H 3700 5100 50  0001 L CNN
+	1    3700 5100
+	0    -1   1    0
+$EndComp
+Wire Wire Line
+	4550 5200 3900 5200
+Wire Wire Line
+	4200 4800 4200 5200
+Connection ~ 4200 5200
+Wire Wire Line
+	3950 4900 3700 4900
+Connection ~ 3300 5200
 $EndSCHEMATC

Commit message: ネットリスト更新 配線編集
Connections:
- net MCU/T15_CH2: now also Q1.2 (S), R5.2; no longer Q18.2 (S), R6.2
- net MCU/T4_CH2: now also Q18.2 (S), R6.2; no longer Q1.2 (S), R5.2
Changed lines of the file:
@@
 F11 "T1_CH2N" O R 6750 3150 60
 F12 "T2_CH1" I L 5750 3250 60
-F13 "T15_CH2" I L 5750 4150 60
+F13 "T15_CH2" I L 5750 4050 60
 F14 "FAULT1" I R 6750 3450 60
 F15 "FAULT2" I R 6750 4500 60
 F16 "LED0" O L 5750 4650 60
 F17 "T8_CH2" O R 6750 4100 60
-F18 "T4_CH2" I L 5750 4050 60
+F18 "T4_CH2" I L 5750 4150 60
 F19 "T8_CH1" O R 6750 3850 60
 F20 "T3_CH2" I L 5750 3750 60
