File: nmkgmmd_v10_brd.sch (KiCad schematic (older format))
At the start: 29 parts, among them J1 CONN_01X05, J10 CONN_01X10, J2 CONN_01X03, J3 CONN_01X03, J4 CONN_01X04, J5 CONN_01X04, J6 CONN_01X04, J7 CONN_01X03, J8 CONN_01X03, J9 CONN_01X10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

Commit message: LEDの抵抗を決めた
Parts:
- R1, R2: value R -> 1k
Changed lines of the file:
@@
 P 2100 3150
 F 0 "R1" V 2180 3150 50  0000 C CNN
-F 1 "R" V 2100 3150 50  0000 C CNN
+F 1 "1k" V 2100 3150 50  0000 C CNN
 F 2 "Resistors_SMD:R_0603" V 2030 3150 50  0001 C CNN
 F 3 "" H 2100 3150 50  0001 C CNN
@@
 P 2400 3150
 F 0 "R2" V 2480 3150 50  0000 C CNN
-F 1 "R" V 2400 3150 50  0000 C CNN
+F 1 "1k" V 2400 3150 50  0000 C CNN
 F 2 "Resistors_SMD:R_0603" V 2330 3150 50  0001 C CNN
 F 3 "" H 2400 3150 50  0001 C CNN
