File: Logic_Power.sch (KiCad schematic (older format))
At the start: 21 parts, among them SW2 SW_DPDT_x2, U2 MCP16301, U3 MCP16301

Commit message: コンデンサのサイズを0805から1206に大きくした
Parts:
- C11, C12: footprint Capacitors_SMD:C_0805 -> Capacitors_SMD:C_1206
Changed lines of the file:
@@
 F 0 "C11" H 4325 3550 50  0000 L CNN
 F 1 "10u" H 4325 3350 50  0000 L CNN
-F 2 "Capacitors_SMD:C_0805" H 4338 3300 50  0001 C CNN
+F 2 "Capacitors_SMD:C_1206" H 4338 3300 50  0001 C CNN
 F 3 "" H 4300 3450 50  0001 C CNN
 	1    4300 3450
@@
 F 0 "C12" H 4325 5400 50  0000 L CNN
 F 1 "10u" H 4325 5200 50  0000 L CNN
-F 2 "Capacitors_SMD:C_0805" H 4338 5150 50  0001 C CNN
+F 2 "Capacitors_SMD:C_1206" H 4338 5150 50  0001 C CNN
 F 3 "" H 4300 5300 50  0001 C CNN
 	1    4300 5300
